File: zigbee_comfospot50.kicad_pcb (KiCad board)
At the start: 2 copper layers, 9 parts, among them J1 690357101472, J2 690368191472, J3 Conn_01x04, SW1 SW_Push, U1 ESP32-H2-WROOM-02C

Commit message: Started routing
Parts:
- added R10: 47k, Resistor_SMD:R_0805_2012Metric, F.Cu at (146.5, 102.9)
- added R11: 47k, Resistor_SMD:R_0805_2012Metric, F.Cu at (144.5, 102.9)
- added R3: 10k, Resistor_SMD:R_0805_2012Metric, F.Cu at (120.0, 114.0)
- added R4: 10k, Resistor_SMD:R_0805_2012Metric, F.Cu at (120.0, 112.0)
- added R5: 47k, Resistor_SMD:R_0805_2012Metric, F.Cu at (138.5, 102.9)
- added R6: 47k, Resistor_SMD:R_0805_2012Metric, F.Cu at (140.5, 102.9)
- added R7: 47k, Resistor_SMD:R_0805_2012Metric, F.Cu at (142.5, 102.9)
- added R8: 47k, Resistor_SMD:R_0805_2012Metric, F.Cu at (150.5, 102.9)
- added R9: 47k, Resistor_SMD:R_0805_2012Metric, F.Cu at (148.5, 102.9)
- added SW2: SW_Push, Button_Switch_SMD:SW_Push_1P1T_NO_CK_KSC7xxJ, F.Cu at (127.5, 111.5)
- J2: value 690368191472 -> 690367191472; footprint local:J_Wurth_WR-MM_690368191472 -> local:J_Wurth_WR-MM_690367191472
- R1: footprint Capacitor_SMD:C_0805_2012Metric -> Resistor_SMD:R_0805_2012Metric
- R2: value 1k -> 10k; footprint Capacitor_SMD:C_0805_2012Metric -> Resistor_SMD:R_0805_2012Metric
- SW1: footprint Button_Switch_THT:SW_PUSH_6mm -> Button_Switch_SMD:SW_Push_1P1T_NO_CK_KSC7xxJ
- moved J3 88.1 mm to (120.0, 98.2)
- moved SW1 79.9 mm to (127.5, 104.0), turned to 180 degrees
- moved C2 77.3 mm to (128.0, 95.5), turned to 90 degrees
- moved C1 75.0 mm to (125.0, 95.5), turned to 90 degrees
- moved R2 71.9 mm to (120.0, 110.0)
- moved R1 66.7 mm to (120.0, 94.0)
- moved U1 35.3 mm to (107.9, 103.4)
- moved J2 17.8 mm to (154.3, 109.0), turned to -90 degrees
- moved J1 16.6 mm to (154.3, 97.5), turned to 90 degrees
Connections:
- J3 pad 2: /RXD -> /TXD
- J3 pad 3: /TXD -> /RXD
- U1 pad 10: unconnected-(U1A-IO12-Pad10) -> /LED_ERR
- U1 pad 11: unconnected-(U1A-IO13-Pad11) -> /LED1
- U1 pad 12: unconnected-(U1A-IO14-Pad12) -> /LED2
- U1 pad 15: unconnected-(U1A-IO22-Pad15) -> /LED3
- U1 pad 20: unconnected-(U1A-IO25-Pad20) -> /LED4
- U1 pad 27: unconnected-(U1A-IO1-Pad27) -> /BTN_MINUS
- U1 pad 28: unconnected-(U1A-IO0-Pad28) -> /BTN_PLUS
- U1 pad 5: unconnected-(U1A-IO10-Pad5) -> /LED_AUTO
- U1 pad 6: unconnected-(U1A-IO11-Pad6) -> /LED_FILTER
- U1 pad 7: unconnected-(U1A-IO8-Pad7) -> /GPIO8_BOOT
- U1 pad 8: unconnected-(U1A-IO9-Pad8) -> /GPIO9_BOOT
Routing:
- net /LED1: track 0.00 -> 19.6 mm
- net /LED3: track 0.00 -> 18.3 mm
- net /LED_AUTO: track 0.00 -> 18.0 mm
- net /LED_ERR: track 0.00 -> 17.4 mm
- net /LED2: track 0.00 -> 13.8 mm
- net /LED_FILTER: track 0.00 -> 12.7 mm
- net /LED4: track 0.00 -> 12.6 mm
Other:
- board outline added: 62 x 26.5 mm

Commit message: ROuted
Parts:
- C1, C2, R1: moved to B.Cu
- moved C2 25.7 mm to (105.5, 108.0)
- moved C1 21.1 mm to (108.0, 108.0)
- moved R1 16.9 mm to (110.5, 108.0), turned to -90 degrees
- turned SW1 to 0 degrees
Connections:
- C1 pad 1: Net-(M1B-3V3) -> Net-(U1B-3V3)
- C2 pad 1: Net-(M1B-3V3) -> Net-(U1B-3V3)
- R1 pad 2: Net-(M1B-3V3) -> Net-(U1B-3V3)
- R2 pad 2: Net-(M1C-EN) -> Net-(U1C-EN)
- SW1 pad 2: Net-(M1C-EN) -> Net-(U1C-EN)
- U1 pad 1: (no net) -> Net-(U1B-3V3)
- U1 pad 11: /LED1 -> /LED4
- U1 pad 12: /LED2 -> /LED3
- U1 pad 13: (no net) -> GND
- U1 pad 14: (no net) -> unconnected-(U1B-VBAT-Pad14)
- U1 pad 15: /LED3 -> /LED2
- U1 pad 16: (no net) -> unconnected-(U1D-NC-Pad16)
- U1 pad 17: (no net) -> unconnected-(U1D-NC-Pad17)
- U1 pad 18: (no net) -> unconnected-(U1D-NC-Pad18)
- U1 pad 19: (no net) -> unconnected-(U1D-NC-Pad19)
- U1 pad 2: (no net) -> Net-(U1C-EN)
- U1 pad 20: /LED4 -> /LED1
- U1 pad 21: (no net) -> /RXD
- U1 pad 22: (no net) -> /TXD
- U1 pad 27: /BTN_MINUS -> /BTN_PLUS
- U1 pad 28: /BTN_PLUS -> /BTN_MINUS
- U1 pad 29: (no net) -> GND
- U1 pad 30: (no net) -> GND
- U1 pad 9: (no net) -> GND
Routing:
- net /BTN_MINUS: track 0.00 -> 57.4 mm
- net /BTN_PLUS: track 0.00 -> 56.0 mm
- net /LED2: track 13.8 -> 56.7 mm, vias 0 -> 2
- net /LED1: track 19.6 -> 60.8 mm, vias 0 -> 2
- net /LED_FILTER: track 12.7 -> 49.4 mm, vias 0 -> 2
- net /LED_AUTO: track 18.0 -> 54.3 mm, vias 0 -> 2
- net /LED3: track 18.3 -> 53.6 mm, vias 0 -> 2
- net /LED4: track 12.6 -> 45.1 mm, vias 0 -> 2
- net Net-(U1C-EN): track 0.00 -> 31.8 mm
- net /LED_ERR: track 17.4 -> 47.6 mm, vias 0 -> 2
- net GND: track 0.00 -> 22.1 mm, vias 0 -> 8
- net /GPIO9_BOOT: track 0.00 -> 20.6 mm
- net /TXD: track 0.00 -> 16.1 mm, vias 0 -> 1
- net /RXD: track 0.00 -> 15.4 mm, vias 0 -> 1
- net Net-(U1B-3V3): track 0.00 -> 11.6 mm, vias 0 -> 1
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- added copper zone on In2.Cu, net +3.3V
- added copper zone on In1.Cu, net GND
Other:
- copper layers 2 -> 4
